File: PWMGenerator-rkroetch1/PWMGenerator-rkroetch1.kicad_sch (KiCad schematic)
At the start: 0 parts

Commit message: PCB Part A done, I think
Parts:
- added C1: 220uF, symbol Device:C_Polarized_US
- added C2: 10uF, symbol Device:C_Polarized_US
- added C3: 0.1uF, symbol Device:C
- added D1, D2, D3, D4, D5: 1N4005, Diode_THT:D_DO-41_SOD81_P10.16mm_Horizontal, symbol Diode:1N4005
- added D6: LED, symbol Device:LED
- added F1: Fuse, symbol Device:Fuse
- added J1: Conn_01x03, symbol Connector_Generic:Conn_01x03
- added Q1, Q2: 2N3904, Package_TO_SOT_THT:TO-92_Inline, symbol Transistor_BJT:2N3904
- added Q3, Q4: 2N3906, Package_TO_SOT_THT:TO-92_Inline, symbol Transistor_BJT:2N3906
- added R1, R8: 2.2k, symbol Device:R_US
- added R10: 8.2k, symbol Device:R_US
- added R11: 180, symbol Device:R_US
- added R2: 1M, symbol Device:R_US
- added R3: 330, symbol Device:R_US
- added R4: 10k, symbol Device:R_US
- added R5: 220k, symbol Device:R_US
- added R6: 390k, symbol Device:R_US
- added R7: 22k, symbol Device:R_US
- added R9: 5k, symbol Device:R_Potentiometer_US
- added SW1: SW_SPST, symbol Switch:SW_SPST
- added U1: LM7805_TO220, Package_TO_SOT_THT:TO-220-3_Vertical, symbol Regulator_Linear:LM7805_TO220
- added U2: LM339AJ, symbol Comparator:LM339
- added V1: VSIN, symbol Simulation_SPICE:VSIN
Connections:
- new net: D1.1 (K), D3.2 (A), F1.2
- new net: F1.1, SW1.2 (B)
- new net: Q1.2 (B), R2.2
- new net: Q1.3 (C), Q2.2 (B), R4.2
- new net: C3.1, Q2.3 (C), Q3.3 (C), U2.4 (-)
- new net: C2.1, J1.1 (Pin_1), Q4.1 (E), R3.1, R4.1, R5.1, R7.1, R8.1, U1.3 (VO), U2.3 (V+)
- new net: Q3.2 (B), R5.2, R6.1
- new net: Q3.1 (E), R7.2
- new net: D3.1 (K), D4.1 (K), D5.2 (A), R1.1, R2.1
- new net: R10.1, U2.2
- new net: R8.2, R9.1, U2.5 (+)
- new net: J1.2 (Pin_2), Q4.3 (C), R11.1
- new net: Q4.2 (B), R10.2
- new net: D6.2 (A), R3.2
- new net GND: C1.2, C2.2, C3.2, D1.2 (A), D2.2 (A), D6.1 (K), J1.3 (Pin_3), Q1.1 (E), Q2.1 (E), R1.2, R11.2, R6.2, R9.2, R9.3, U1.2 (GND), U2.12 (V-)
- new net GNDPWR: D2.1 (K), D4.2 (A), V1.2
- new net VAC: SW1.1 (A), V1.1
- new net VCC: C1.1, D5.1 (K), U1.1 (VI)
Other:
- company: (none) -> NAIT CNT
- title: (none) -> CMPE2150 PWM Generator - rkroetch1

Commit message: PCB Part B Part 2
Parts:
- C1: footprint (none) -> Capacitor_THT:CP_Radial_D8.0mm_P3.50mm
- C2: footprint (none) -> Capacitor_THT:CP_Radial_D10.0mm_P5.00mm
- C3: footprint (none) -> Capacitor_SMD:C_0805_2012Metric
- D1, D2, D3, D4, D5: value 1N4005 -> 1N4005G; footprint Diode_THT:D_DO-41_SOD81_P10.16mm_Horizontal -> Diode_SMD:D_0805_2012Metric
- D6: value LED -> LED_GREEN; footprint (none) -> LED_THT:LED_D5.0mm_GREEN
- F1: value Fuse -> NANOSMDC016F-2; footprint (none) -> NANOSMDC016F-2:RESC3115X65N; symbol Device:Fuse -> NANOSMDC016F-2:NANOSMDC016F-2
- J1: value Conn_01x03 -> Conn_01x03_Pin; footprint (none) -> Connector_PinHeader_2.54mm:PinHeader_1x03_P2.54mm_Vertical
- Q1, Q2, Q3, Q4: footprint Package_TO_SOT_THT:TO-92_Inline -> Package_TO_SOT_SMD:SOT-23
- R1, R10, R11, R2, R3, R4, R5, R6, R7, R8: footprint (none) -> Resistor_SMD:R_0805_2012Metric
- R9: footprint (none) -> Potentiometer_THT:Potentiometer_Piher_PT-15-V15_Vertical_Hole
- SW1: value SW_SPST -> AS11CP; footprint (none) -> AS11CP:SW_AS11CP; symbol Switch:SW_SPST -> AS11CP:AS11CP; MANUFACTURER (none) -> NKK Switches; PARTREV (none) -> N/A; STANDARD (none) -> Manufacturer Recommendations
- U2: footprint (none) -> Package_SO:SOIC-14_3.9x8.7mm_P1.27mm
- V1: value VSIN -> Barrel_Jack; footprint (none) -> Connector_BarrelJack:BarrelJack_Horizontal; symbol Simulation_SPICE:VSIN -> Connector:Barrel_Jack
Connections:
- net at F1.1: now also SW1.3; no longer SW1.2 (B)
- net VAC: no longer names the net of SW1.1, V1.1
Other:
- moved on the sheet: C1, C2, C3, D1, D2, D3, D4, D5, D6, J1, Q1, Q2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

Commit message: PCB Part B Part 3
Parts:
- added unit 2 of U2
- added unit 3 of U2
- added unit 4 of U2
- D1, D2, D3, D4, D5: footprint Diode_SMD:D_0805_2012Metric -> Diode_THT:D_DO-41_SOD81_P10.16mm_Horizontal
- D6: footprint LED_THT:LED_D5.0mm_GREEN -> LED_THT:LED_D5.0mm
- F1: footprint NANOSMDC016F-2:RESC3115X65N -> Library:RESC3115X65N
- Q1, Q2, Q3, Q4: footprint Package_TO_SOT_SMD:SOT-23 -> Package_TO_SOT_THT:TO-92_Inline
- SW1: footprint AS11CP:SW_AS11CP -> Library:SW_AS11CP
Connections:
- net VCC: now also U2.3 (V+)
- net at C2.1, J1.1 (Pin_1), Q4.1 (E)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: no longer U2.3 (V+)
- no-connect marks 0 -> 9

Commit message: Update Jack footprint, finish part 2
Parts:
- V1: footprint Connector_BarrelJack:BarrelJack_Horizontal -> Connector_BarrelJack:BarrelJack_SwitchcraftConxall_RAPC10U_Horizontal
Changed lines of the file:
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@@
 		(title "CMPE2150 PWM Generator - rkroetch1")
 		(date "2025-12-12")
-		(rev "2")
+		(rev "2.1")
 		(company "NAIT CNT")
 		(comment 1 "Robert Kroetch")
@@
 			)
 		)
-		(property "Footprint" "Connector_BarrelJack:BarrelJack_Horizontal"
+		(property "Footprint" "Connector_BarrelJack:BarrelJack_SwitchcraftConxall_RAPC10U_Horizontal"
 			(at 20.32 50.546 0)
 			(effects
